File: test1.kicad_pcb (KiCad board)
At the start: 2 copper layers, 22 parts, among them P1 Conn_01x03, P2 Conn_01x02, P3 Conn_01x04, U1 L78L05_TO92, U2 LM339

Commit message: Add files via upload
Parts:
- moved C5 83.2 mm to (144.5, 76.4)
- moved C6 81.4 mm to (144.0, 84.0)
- moved R2 81.3 mm to (154.9, 68.6), turned to 0 degrees
- moved R7 75.0 mm to (175.3, 73.7), turned to -90 degrees
- moved C1 73.1 mm to (135.5, 69.1)
- moved C2 73.1 mm to (135.5, 74.1)
- moved C3 73.1 mm to (135.5, 79.2)
- moved P3 69.6 mm to (136.0, 94.2), turned to 0 degrees
- moved R1 68.4 mm to (170.2, 68.6), turned to 0 degrees
- moved R5 68.0 mm to (121.9, 84.8), turned to 0 degrees
- moved R4 67.6 mm to (121.9, 80.7), turned to 0 degrees
- moved C7 66.4 mm to (157.6, 73.7), turned to 0 degrees
- moved R6 65.3 mm to (180.3, 83.8), turned to 90 degrees
- moved P2 63.6 mm to (145.3, 94.0), turned to 0 degrees
- moved C4 62.7 mm to (165.1, 58.4)
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Routing:
- net Net-(P3-Pin_2): track 110.3 -> 0.00 mm
- net Net-(P1-Pin_1): track 132.6 -> 30.6 mm
- net GND: track 121.5 -> 54.2 mm
- net Net-(C1-Pad1): track 64.7 -> 0.00 mm
- net Net-(U2B-+): track 63.7 -> 5.08 mm, vias 1 -> 0
- net Net-(U2A--): track 47.0 -> 5.16 mm
- net Net-(U2A-+): track 41.6 -> 0.00 mm
- net Net-(P3-Pin_3): track 38.6 -> 0.38 mm
- net Net-(P1-Pin_3): track 25.4 -> 0.00 mm
- net Net-(U2C-+): track 25.0 -> 5.08 mm
Other:
- board outline added: 30.5 x 66 mm

Commit message: update
Parts:
- moved R4 65.1 mm to (184.4, 99.1), turned to -90 degrees
- moved R5 60.2 mm to (180.3, 99.1), turned to -90 degrees
- moved C5 54.1 mm to (180.4, 116.8)
- moved C1 51.3 mm to (175.2, 101.6), turned to 180 degrees
- moved C2 45.6 mm to (175.2, 96.5), turned to 180 degrees
- moved C3 41.5 mm to (175.2, 91.5), turned to 180 degrees
- moved R9 38.8 mm to (160.0, 94.0), turned to -90 degrees
- moved C6 36.5 mm to (170.3, 109.2)
- moved R10 35.8 mm to (156.0, 94.0), turned to -90 degrees
- moved R3 35.2 mm to (154.9, 88.9)
- moved P2 35.1 mm to (180.3, 93.5), turned to 90 degrees
- moved P3 26.2 mm to (157.5, 109.2), turned to 90 degrees
- moved U1 6.35 mm to (165.1, 58.4)
- moved C4 5.12 mm to (160.0, 58.4)
- moved P1 3.59 mm to (172.7, 61.0), turned to 180 degrees
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Routing:
- net GND: track 54.2 -> 0.00 mm
- net Net-(P1-Pin_1): track 30.6 -> 0.00 mm
- net Net-(U2C-+): track 5.08 -> 0.00 mm
- net Net-(U2A--): track 5.16 -> 0.08 mm
- net Net-(U2B-+): track 5.08 -> 0.00 mm
Other:
- board size 30.5 x 66 mm -> 35.6 x 71.1 mm

Commit message: dalawa nalang
Parts:
- moved C4 78.9 mm to (165.1, 137.2)
- moved C5 56.2 mm to (162.6, 63.5)
- moved U1 49.9 mm to (152.4, 106.7), turned to 180 degrees
- moved C7 40.7 mm to (157.5, 114.4), turned to -90 degrees
- moved P2 39.9 mm to (167.2, 55.9), turned to 180 degrees
- moved C3 38.8 mm to (167.6, 129.5)
- moved C2 28.9 mm to (167.6, 124.5)
- moved R7 25.9 mm to (170.2, 99.1), turned to 180 degrees
- moved R6 22.7 mm to (160.0, 94.0), turned to 0 degrees
- moved U2 20.4 mm to (142.3, 91.4), turned to 180 degrees
- moved R8 20.3 mm to (170.2, 104.1), turned to 180 degrees
- moved C1 19.3 mm to (167.6, 119.4)
- moved R4 19.1 mm to (170.2, 86.4), turned to 180 degrees
- moved R1 17.8 mm to (152.4, 68.6), turned to 90 degrees
- moved R2 17.0 mm to (170.2, 76.2), turned to 180 degrees
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Routing:
- net GND: track 0.00 -> 263.9 mm
- net Net-(P1-Pin_1): track 0.00 -> 229.0 mm
- net Net-(C1-Pad1): track 0.00 -> 106.2 mm
- net Net-(U2B-+): track 0.00 -> 75.3 mm
- net Net-(U2A-+): track 0.00 -> 66.4 mm
- net Net-(U2C-+): track 0.00 -> 66.1 mm
- net Net-(P3-Pin_3): track 0.00 -> 64.6 mm
- net Net-(P3-Pin_2): track 0.00 -> 63.3 mm
- net Net-(U2A--): track 0.08 -> 38.6 mm
- net Net-(P1-Pin_3): track 0.00 -> 35.7 mm
Other:
- board size 35.6 x 71.1 mm -> 43.2 x 91.4 mm

Commit message: may dalawang jumper ;-;
Connections:
- C1 pad 1: Net-(C1-Pad1) -> GND
- C2 pad 1: Net-(C1-Pad1) -> GND
- C3 pad 1: Net-(C1-Pad1) -> GND
- R3 pad 1: Net-(C1-Pad1) -> GND
- U2 pad 13: unconnected-(U2-Pad13) -> GND
- U2 pad 14: Net-(C1-Pad1) -> GND
Routing:
- net Net-(C1-Pad1): track 106.2 -> 0.00 mm
- net GND: track 263.9 -> 368.9 mm
- net Net-(U2A--): track 38.6 -> 70.5 mm
- net Net-(U2A-+): track 66.4 -> 97.4 mm
- net Net-(P1-Pin_1): track 229.0 -> 253.9 mm
- net Net-(P3-Pin_2): track 63.3 -> 70.8 mm
- net Net-(P3-Pin_3): track 64.6 -> 67.1 mm
Other:
- board size 43.2 x 91.4 mm -> 45.7 x 91.4 mm
