File: FinalProject.kicad_pcb (KiCad board)
At the start: 2 copper layers, 22 parts, among them P1 Conn_01x03, P2 Conn_01x02, P3 Conn_01x04, U1 L78L05_TO92, U2 LM339

Commit message: commit
Parts:
- moved P2 90.8 mm to (167.2, 55.9), turned to 180 degrees
- moved C5 87.6 mm to (162.6, 63.5)
- moved R1 79.1 mm to (152.4, 68.6), turned to 90 degrees
- moved R2 66.2 mm to (170.2, 76.2)
- moved R6 64.1 mm to (160.0, 94.0)
- moved U2 56.8 mm to (142.3, 91.4), turned to 180 degrees
- moved R7 55.9 mm to (170.2, 99.1)
- moved P1 51.4 mm to (162.6, 71.1), turned to 90 degrees
- moved C7 46.3 mm to (157.5, 114.4), turned to -90 degrees
- moved C6 45.8 mm to (162.6, 114.3)
- moved P3 43.4 mm to (162.6, 109.2), turned to 90 degrees
- moved R10 43.4 mm to (152.4, 86.4)
- moved R9 43.2 mm to (148.8, 86.4)
- moved R8 41.7 mm to (170.2, 104.1), turned to 180 degrees
- moved C4 41.6 mm to (165.1, 137.2)
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Connections:
- C1 pad 1: Net-(C1-Pad1) -> GND
- C2 pad 1: Net-(C1-Pad1) -> GND
- C3 pad 1: Net-(C1-Pad1) -> GND
- R3 pad 1: Net-(C1-Pad1) -> GND
- U2 pad 13: unconnected-(U2-Pad13) -> GND
- U2 pad 14: Net-(C1-Pad1) -> GND
Routing:
- net GND: track 121.5 -> 368.9 mm
- net Net-(P1-Pin_1): track 132.6 -> 253.9 mm
- net Net-(C1-Pad1): track 64.7 -> 0.00 mm
- net Net-(U2A-+): track 41.6 -> 97.4 mm
- net Net-(U2C-+): track 25.0 -> 66.1 mm
- net Net-(P3-Pin_2): track 110.3 -> 70.8 mm
- net Net-(P3-Pin_3): track 38.6 -> 70.5 mm
- net Net-(U2A--): track 47.0 -> 70.5 mm
- net Net-(U2B-+): track 63.7 -> 75.3 mm, vias 1 -> 0
- net Net-(P1-Pin_3): track 25.4 -> 35.7 mm
Other:
- board outline added: 45.7 x 91.4 mm

Commit message: added jumpers to pcb
Parts:
- moved U1 5.08 mm to (147.3, 106.7)
Routing:
- net Net-(U2A--): track 70.5 -> 46.8 mm, vias 0 -> 2
- net Net-(U2A-+): track 97.4 -> 74.4 mm, vias 0 -> 2
- net GND: track 368.9 -> 377.1 mm
- net Net-(P3-Pin_2): track 70.8 -> 72.9 mm
- net Net-(P3-Pin_3): track 70.5 -> 72.6 mm
Other:
- board size 45.7 x 91.4 mm -> 48.3 x 91.4 mm

Commit message: changed file names and deleted previous version
Parts:
- moved C3 72.2 mm to (144.9, 61.0), turned to 0 degrees
- moved R2 59.1 mm to (166.1, 135.2), turned to 90 degrees
- moved C2 55.7 mm to (139.8, 76.2), turned to 0 degrees
- moved C1 55.6 mm to (144.9, 68.6), turned to 0 degrees
- moved R1 55.6 mm to (166.1, 122.5)
- moved C7 54.5 mm to (161.9, 60.1), turned to 90 degrees
- moved P1 51.2 mm to (148.8, 120.4), turned to 0 degrees
- moved C6 49.7 mm to (172.1, 65.5)
- moved U2 35.2 mm to (158.0, 123.0), turned to -90 degrees
- moved R5 30.6 mm to (139.7, 93.0), turned to 90 degrees
- moved U1 29.4 mm to (162.0, 132.1)
- moved R4 23.0 mm to (148.2, 93.0), turned to 90 degrees
- moved R9 22.7 mm to (170.2, 94.0)
- moved R8 21.4 mm to (148.8, 105.2), turned to 0 degrees
- moved R3 20.5 mm to (177.8, 91.4), turned to 90 degrees
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Routing:
- net GND: track 377.1 -> 225.0 mm
- net Net-(U2C-+): track 66.1 -> 18.2 mm
- net Net-(P3-Pin_2): track 72.9 -> 41.7 mm
- net Net-(P1-Pin_3): track 35.7 -> 9.47 mm
- net Net-(U2B-+): track 75.3 -> 52.8 mm
- net Net-(U2A--): track 46.8 -> 67.1 mm, vias 2 -> 0
- net Net-(U2A-+): track 74.4 -> 88.9 mm, vias 2 -> 0
- net Net-(P3-Pin_3): track 72.6 -> 60.5 mm
- net Net-(P1-Pin_1): track 253.9 -> 260.4 mm
Other:
- board size 48.3 x 91.4 mm -> 50.8 x 94 mm
